Commit message: usdaFile

File: src/RLforHexapod/assets/urdf/robot.urdf (robot description, URDF)
Before this commit: robot HexapodRobot, 25 links, 24 joints
Links:
- link body: geometry collision mesh filename=C:\Users\COM\isaac-lab-workspace\RLForHexapod\src\RLforHexa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; collision mesh filename=C:\Users\COM\isaac-lab-workspace\RLForHexapod\src\RLforHexa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
- link coxa: geometry collision mesh filename=C:\Users\COM\isaac-lab-workspace\RLForHexapod\src\RLforHexa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; collision mesh filename=C:\Users\COM\isaac-lab-workspace\RLForHexapod\src\RLforHexa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
- link coxa_2: geometry collision mesh filename=C:\Users\COM\isaac-lab-workspace\RLForHexapod\src\RLforHexa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; collision mesh filename=C:\Users\COM\isaac-lab-workspace\RLForHexapod\src\RLforHexa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
- link coxa_3: geometry collision mesh filename=C:\Users\COM\isaac-lab-workspace\RLForHexapod\src\RLforHexa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; collision mesh filename=C:\Users\COM\isaac-lab-workspace\RLForHexapod\src\RLforHexa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
- link coxa_4: geometry collision mesh filename=C:\Users\COM\isaac-lab-workspace\RLForHexapod\src\RLforHexa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; collision mesh filename=C:\Users\COM\isaac-lab-workspace\RLForHexapod\src\RLforHexa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
- link coxa_5: geometry collision mesh filename=C:\Users\COM\isaac-lab-workspace\RLForHexapod\src\RLforHexa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; collision mesh filename=C:\Users\COM\isaac-lab-workspace\RLForHexapod\src\RLforHexa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
- link coxa_6: geometry collision mesh filename=C:\Users\COM\isaac-lab-workspace\RLForHexapod\src\RLforHexa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; collision mesh filename=C:\Users\COM\isaac-lab-workspace\RLForHexapod\src\RLforHexa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
- link femur: geometry collision mesh filename=C:\Users\COM\isaac-lab-workspace\RLForHexapod\src\RLforHexa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; collision mesh filename=C:\Users\COM\isaac-lab-workspace\RLForHexapod\src\RLforHexa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
- link femur_2: geometry collision mesh filename=C:\Users\COM\isaac-lab-workspace\RLForHexapod\src\RLforHexa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; collision mesh filename=C:\Users\COM\isaac-lab-workspace\RLForHexapod\src\RLforHexa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
- link femur_3: geometry collision mesh filename=C:\Users\COM\isaac-lab-workspace\RLForHexapod\src\RLforHexa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; collision mesh filename=C:\Users\COM\isaac-lab-workspace\RLForHexapod\src\RLforHexa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
- link femur_4: geometry collision mesh filename=C:\Users\COM\isaac-lab-workspace\RLForHexapod\src\RLforHexa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; collision mesh filename=C:\Users\COM\isaac-lab-workspace\RLForHexapod\src\RLforHexa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
- link femur_5: geometry collision mesh filename=C:\Users\COM\isaac-lab-workspace\RLForHexapod\src\RLforHexa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; collision mesh filename=C:\Users\COM\isaac-lab-workspace\RLForHexapod\src\RLforHexa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
- link femur_6: geometry collision mesh filename=C:\Users\COM\isaac-lab-workspace\RLForHexapod\src\RLforHexa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; collision mesh filename=C:\Users\COM\isaac-lab-workspace\RLForHexapod\src\RLforHexa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
- link tibia: geometry collision mesh filename=C:\Users\COM\isaac-lab-workspace\RLForHexapod\src\RLforHexa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; collision mesh filename=C:\Users\COM\isaac-lab-workspace\RLForHexapod\src\RLforHexa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
- link tibia_2: geometry collision mesh filename=C:\Users\COM\isaac-lab-workspace\RLForHexapod\src\RLforHexa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; collision mesh filename=C:\Users\COM\isaac-lab-workspace\RLForHexapod\src\RLforHexa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
- link tibia_3: geometry collision mesh filename=C:\Users\COM\isaac-lab-workspace\RLForHexapod\src\RLforHexa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; collision mesh filename=C:\Users\COM\isaac-lab-workspace\RLForHexapod\src\RLforHexa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
- link tibia_4: geometry collision mesh filename=C:\Users\COM\isaac-lab-workspace\RLForHexapod\src\RLforHexa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; collision mesh filename=C:\Users\COM\isaac-lab-workspace\RLForHexapod\src\RLforHexa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
- link tibia_5: geometry collision mesh filename=C:\Users\COM\isaac-lab-workspace\RLForHexapod\src\RLforHexa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; collision mesh filename=C:\Users\COM\isaac-lab-workspace\RLForHexapod\src\RLforHexa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
- link tibia_6: geometry collision mesh filename=C:\Users\COM\isaac-lab-workspace\RLForHexapod\src\RLforHexa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; collision mesh filename=C:\Users\COM\isaac-lab-workspace\RLForHexapod\src\RLforHexa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

Commit message: realrobotUrdf

File: src/RLforHexapod/assets/urdf/robot.urdf (robot description, URDF)
Before this commit: robot HexapodRobot, 25 links, 24 joints
Links:
- removed link L1_feet
- removed link L2_feet
- removed link L3_feet
- removed link L4_feet
- removed link L5_feet
- removed link L6_feet
- link body: geometry collision mesh filename=package://assets/battery.stl; collision mesh filename=package://assets/batterycover.stl
- link coxa: geometry collision mesh filename=package://assets/coxajoint.stl; collision mesh filename=package://assets/motorhorn.stl
- link coxa_2: geometry collision mesh filename=package://assets/coxajoint.stl; collision mesh filename=package://assets/motorhorn.stl
- link coxa_3: geometry collision mesh filename=package://assets/coxajoint.stl; collision mesh filename=package://assets/motorhorn.stl
- link coxa_4: geometry collision mesh filename=package://assets/coxajoint.stl; collision mesh filename=package://assets/motorhorn.stl
- link coxa_5: geometry collision mesh filename=package://assets/coxajoint.stl; collision mesh filename=package://assets/motorhorn.stl
- link coxa_6: geometry collision mesh filename=package://assets/coxajoint.stl; collision mesh filename=package://assets/motorhorn.stl
- link femur: geometry collision mesh filename=package://assets/femur.stl; collision mesh filename=package://assets/jointcover.stl
- link femur_2: geometry collision mesh filename=package://assets/femur.stl; collision mesh filename=package://assets/jointcover.stl
- link femur_3: geometry collision mesh filename=package://assets/femur.stl; collision mesh filename=package://assets/jointcover.stl
- link femur_4: geometry collision mesh filename=package://assets/femur.stl; collision mesh filename=package://assets/jointcover.stl
- link femur_5: geometry collision mesh filename=package://assets/femur.stl; collision mesh filename=package://assets/jointcover.stl
- link femur_6: geometry collision mesh filename=package://assets/femur.stl; collision mesh filename=package://assets/jointcover.stl
- link tibia: geometry collision mesh filename=package://assets/rc9mg.stl; collision mesh filename=package://assets/tibia.stl
- link tibia_2: geometry collision mesh filename=package://assets/rc9mg.stl; collision mesh filename=package://assets/tibia.stl
- link tibia_3: geometry collision mesh filename=package://assets/rc9mg.stl; collision mesh filename=package://assets/tibia.stl
- link tibia_4: geometry collision mesh filename=package://assets/rc9mg.stl; collision mesh filename=package://assets/tibia.stl
- link tibia_5: geometry collision mesh filename=package://assets/rc9mg.stl; collision mesh filename=package://assets/tibia.stl
- link tibia_6: geometry collision mesh filename=package://assets/rc9mg.stl; collision mesh filename=package://assets/tibia.stl
Joints:
- removed joint L1_feet_frame
- removed joint L2_feet_frame
- removed joint L3_feet_frame
- removed joint L4_feet_frame
- removed joint L5_feet_frame
- removed joint L6_feet_frame

Commit message: update12

File: src/RLforHexapod/assets/urdf/robot.urdf (robot description, URDF)
Before this commit: robot HexapodRobot, 19 links, 18 joints
Joints:
- joint L1_femur: limit lower=0 upper=3.14159 effort=1.8633 velocity=6.545 -> lower=0 upper=4.71239 effort=1.8633 velocity=6.545
- joint L1_tibia: limit lower=-3.14159 upper=0 effort=1.8633 velocity=6.545 -> lower=-4.71239 upper=0 effort=1.8633 velocity=6.545
- joint L2_femur: limit lower=0 upper=3.14159 effort=1.8633 velocity=6.545 -> lower=0 upper=4.71239 effort=1.8633 velocity=6.545
- joint L2_tibia: limit lower=-3.14159 upper=0 effort=1.8633 velocity=6.545 -> lower=-4.71239 upper=0 effort=1.8633 velocity=6.545
- joint L3_femur: limit lower=0 upper=3.14159 effort=1.8633 velocity=6.545 -> lower=0 upper=4.71239 effort=1.8633 velocity=6.545
- joint L3_tibia: limit lower=-3.14159 upper=0 effort=1.8633 velocity=6.545 -> lower=-4.71239 upper=0 effort=1.8633 velocity=6.545
- joint L4_femur: limit lower=0 upper=3.14159 effort=1.8633 velocity=6.545 -> lower=0 upper=4.71239 effort=1.8633 velocity=6.545
- joint L4_tibia: limit lower=-3.14159 upper=0 effort=1.8633 velocity=6.545 -> lower=-4.71239 upper=0 effort=1.8633 velocity=6.545
- joint L5_femur: limit lower=0 upper=3.14159 effort=1.8633 velocity=6.545 -> lower=0 upper=4.71239 effort=1.8633 velocity=6.545
- joint L5_tibia: limit lower=-3.14159 upper=0 effort=1.8633 velocity=6.545 -> lower=-4.71239 upper=0 effort=1.8633 velocity=6.545
- joint L6_femur: limit lower=0 upper=3.14159 effort=1.8633 velocity=6.545 -> lower=0 upper=4.71239 effort=1.8633 velocity=6.545
- joint L6_tibia: limit lower=-3.14159 upper=0 effort=1.8633 velocity=6.545 -> lower=-4.71239 upper=0 effort=1.8633 velocity=6.545
